File: HPS-Rect-Clock/HPS-Rect-Clock.kicad_sch (KiCad schematic)
At the start: 4 parts

Commit message: Week 1 Schematics
Parts:
- added C? (x6): C_0805_10uf, footprints:C_0805_2012Metric, symbol HPS:C_0805_10uf
- added C? (x2): C_0805_0.1uf, footprints:C_0805_2012Metric, symbol HPS:C_0805_0.1uf
- added D?: LED_0805, footprints:LED_0805_2012Metric, symbol HPS:LED_0805
- added J?: PJ-102AH, footprints:PJ-102AH, symbol HPS:PJ-102AH
- added J?: Conn_01x06, footprints:PinHeader_1x06_P2.54mm_Vertical, symbol HPS:Conn_01x06
- added R?: R_0805_2.2K, footprints:R_0805_2012Metric, symbol HPS:R_0805_2.2K
- added R?: R_0805_10K, footprints:R_0805_2012Metric, symbol HPS:R_0805_10K
- added U?: ATmega328-PU, footprints:DIP-28_W7.62mm, symbol HPS:ATmega328-PU
- added Y1: Crystal_16MHz, footprints:Crystal_SMD_HC49-SD, symbol HPS:Crystal_16MHz
Connections:
- new net: C?.2, J?.1 (POLE)
- new net: C?.1, R?.2, U?.1 (~{RESET}/PC6)
- new net: C?.1, U?.21 (AREF)
- new net: C?.1, C?.1, U?.10 (XTAL2/PB7), U?.9 (XTAL1/PB6), Y1.1, Y1.2
- new net: J?.4 (Pin_4), U?.2 (PD0)
- new net: J?.5 (Pin_5), U?.3 (PD1)
- new net: D?.2 (A), R?.2
- new net GND: C?.1, C?.2, C?.2, C?.2, C?.2, C?.2, C?.2, D?.1 (K), J?.1 (Pin_1), J?.2 (OUT), J?.2 (Pin_2)
- new net LED_SCK: R?.1, U?.19 (PB5)
- new net RTS: C?.2, J?.6 (Pin_6)
- new net VCC: C?.1, C?.1, C?.1, R?.1, U?.20 (AVCC), U?.7 (VCC)
- no-connect marks 0 -> 2

Commit message: Week 2
Parts:
- removed C? (x3): C_0805_10uf, footprints:C_0805_2012Metric, symbol HPS:C_0805_10uf
- removed C?: C_0805_0.1uf, footprints:C_0805_2012Metric, symbol HPS:C_0805_0.1uf
- added C2: C_0805_0.1uf, footprints:C_0805_2012Metric, symbol HPS:C_0805_10uf
- added C3: C_0805_0.1uf, footprints:C_0805_2012Metric, symbol HPS:C_0805_0.1uf
- added C7: C_0805_0.11uf, footprints:C_0805_2012Metric, symbol HPS:C_0805_0.1uf
- added R? (x2): R_0805_4.7K, footprints:R_0805_2012Metric, symbol HPS:R_0805_4.7K
- added SW?: Omron_B3F_SPST, footprints:SW_SPST_Omron_B3FS-100xP, symbol HPS:Omron_B3F_SPST
- added U?: L7805_TO92, footprints:TO-92_Inline, symbol HPS:L7805_TO92
- C1: renamed from C?; value C_0805_10uf -> C_0805_0.1uf
- C4, C5: renamed from C?; value C_0805_10uf -> C_0805_22pf
- C6: renamed from C?; value C_0805_0.1uf -> C_0805_1uf
- gave numbers to parts that had none: 5
Connections:
- net GND: now also R1.2, U?.22 (GND), U?.8 (GND), C2.2, C7.1, SW?.1 (A), SW?.2 (A), U?.2 (GND); no longer D1.1 (K)
- net LED_SCK: now also D1.2 (A); no longer R1.1
- net VCC: now also C2.1, C7.2, U?.1 (VO)
- net at C6.2, J2.1 (POLE): now also U?.3 (VI)
- net RESET: now reaches R2.2, U?.1 (~{RESET}/PC6)
- net RESET: now also C3.1, SW?.3 (B), SW?.4 (B)
- net at C4.1, U?.9 (XTAL1/PB6), Y1.1: no longer C5.1, U?.10 (XTAL2/PB7), Y1.2
- net at J1.4 (Pin_4): now also R?.1; no longer U?.2 (PD0)
- net at J1.5 (Pin_5): now also R?.1; no longer U?.3 (PD1)
- net RTS: no longer names the net of J1.6 (Pin_6)
- net RTS: now also C3.2
- new net: C5.1, U?.10 (XTAL2/PB7), Y1.2
- new net: D1.1 (K), R1.1
- new net RXD: R?.2, U?.2 (PD0)
- new net TXD: R?.2, U?.3 (PD1)
Other:
- note added: "LED"
- note added: "MCU"
- note added: "Power Input"
- note added: "Serial"
- note added: "Vf = 2v Vr = 3v 10mcd @ 1.35mA therefor R = 2.2KOhm"
- moved on the sheet: C1, C4, C5, C6, D1, H1, H2, H3, H4, J1, J2, R1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

Commit message: Week 3
Other:
- note added: "Crystal Rectangular Schematic"
Changed lines of the file:
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@@
     (stroke (width 0) (type default) (color 0 0 0 0))
+  )
+  (text "Crystal Rectangular Schematic\n" (at 186.69 190.5 0)
+    (effects (font (size 1.27 1.27)) (justify left bottom))
   )
   (text "MCU" (at 124.46 123.19 0)

Commit message: Week 3
Parts:
- removed H1, H2, H3, H4: MountingHole, footprints:MountingHole_3.2mm_M3, symbol HPS:MountingHole
- added D? (x13): NEOPIXEL_SMT, footprints:LED_SK6812_PLCC4_5.0x5.0mm_P3.2mm, symbol HPS:NEOPIXEL_SMT
- added DS?: TC1602A-01T, footprints:TC1602A-01T, symbol HPS:TC1602A-01T
- added R?: R_0805_47, footprints:R_0805_2012Metric, symbol HPS:R_0805_47
Connections:
- net GND: now also C4.1, C5.1, U?.10 (XTAL2/PB7), U?.9 (XTAL1/PB6), Y1.1, Y1.2, D?.1 (VSS), D?.1 (VSS), D?.1 (VSS), D?.1 (VSS), D?.1 (VSS), D?.1 (VSS), D?.1 (VSS), D?.1 (VSS), D?.1 (VSS), D?.1 (VSS), D?.1 (VSS), D?.1 (VSS), D?.1 (VSS), DS?.1 (VSS)
- net LED_SCK: now also U?.18 (PB4), DS?.8 (D1)
- net VCC: now also D?.2 (DIN), D?.3 (VDD), D?.3 (VDD), D?.3 (VDD), D?.3 (VDD), D?.3 (VDD), D?.3 (VDD), D?.3 (VDD), D?.3 (VDD), D?.3 (VDD), D?.3 (VDD), D?.3 (VDD), D?.3 (VDD), D?.3 (VDD), D?.4 (DOUT), DS?.3 (VO)
- net at U?.13 (PD7): now also R?.1
- net at U?.14 (PB0): now also DS?.6 (E)
- net at U?.15 (PB1): now also DS?.5 (R/W)
- net at U?.16 (PB2): now also DS?.4 (RS)
- net at U?.17 (PB3): now also DS?.7 (D0)
- net at U?.23 (PC0): now also DS?.9 (D2)
- net at U?.24 (PC1): now also DS?.10 (D3)
- net at U?.25 (PC2): now also DS?.11 (D4)
- net at U?.4 (PD2): now also DS?.12 (D5)
- net at U?.5 (PD3): now also DS?.13 (D6)
- net at U?.6 (PD4): now also DS?.14 (D7)
- new net: D?.2 (DIN), D?.4 (DOUT) (x11)
- new net: D?.2 (DIN), R?.2
Other:
- moved on the sheet: C1, C2, C3, C4, C5, C6, C7, J1, J2, R2, R?, SW?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

Commit message: Week 4
Parts:
- added SW? (x4): Omron_B3F_SPST, footprints:SW_SPST_Omron_B3FS-100xP, symbol HPS:Omron_B3F_SPST
- added U?: DS1307_DIP-8, footprints:DIP-8_W7.62mm, symbol HPS:DS1307_DIP-8
Connections:
- net GND: now also SW?.3 (B), SW?.3 (B), SW?.3 (B), SW?.3 (B), U?.4 (GND)
- net VCC: now also U?.26 (PC3), SW?.1 (A), U?.8 (VCC)
- net at U?.11 (PD5): now also SW?.1 (A)
- net at U?.12 (PD6): now also SW?.1 (A)
- net at U?.27 (PC4): now also SW?.1 (A)

Commit message: Week 5
Parts:
- removed D? (x7): NEOPIXEL_SMT, footprints:LED_SK6812_PLCC4_5.0x5.0mm_P3.2mm, symbol HPS:NEOPIXEL_SMT
- removed U?: L7805_TO92, footprints:TO-92_Inline, symbol HPS:L7805_TO92
- added BT1: Battery_Cell, footprints:BatteryHolder_Keystone_106_1x20mm, symbol HPS:Battery_Cell
- added D10, D11, D12, D13, D6, D7, D8: NEOPIXEL_SMT, footprints:LED_SK6812_PLCC4_5.0x5.0mm_P3.2mm, symbol HPS:NEOPIXEL_SMT
- added R10, R7, R8, R9: R_0805_10K, footprints:R_0805_2012Metric, symbol HPS:R_0805_10K
- added R11, R12: R_0805_4.7K, footprints:R_0805_2012Metric, symbol HPS:R_0805_4.7K
- added R6: R_0805_47, footprints:R_0805_2012Metric, symbol HPS:R_0805_47
- added RV1: R_POT_10K, footprints:Potentiometer_Bourns_3386P_Vertical, symbol HPS:R_POT_10K
- added U?: L7805, symbol HPS:L7805
- added Y2: Crystal_32768Hz, footprints:Crystal_SMD_2Pin_3.2x1.5mm, symbol HPS:Crystal_32768Hz
- gave numbers to parts that had none: 17
Connections:
- net GND: now also DS1.16 (LED(-)), BT1.2 (-), D10.1 (VSS), D11.1 (VSS), D12.1 (VSS), D13.1 (VSS), D6.1 (VSS), D7.1 (VSS), D8.1 (VSS), RV1.1, U?.2 (GND); no longer C4.1, C5.1, U2.10 (XTAL2/PB7), U2.9 (XTAL1/PB6), Y1.1, Y1.2
- net LED_SCK: now also U2.4 (PD2); no longer DS1.8 (D1), U2.18 (PB4), U2.19 (PB5)
- net VCC: now also DS1.2 (VDD), D10.3 (VDD), D11.3 (VDD), D12.3 (VDD), D13.3 (VDD), D6.3 (VDD), D7.3 (VDD), D8.3 (VDD), R10.1, R11.1, R12.1, R6.2, R7.1, R8.1, R9.1, RV1.3, U?.3 (OUT); no longer DS1.3 (VO), SW1.1 (A), U2.26 (PC3)
- net at C6.2, J2.1 (POLE): now also U?.1 (IN)
- net at DS1.10 (D3): no longer U2.24 (PC1)
- net at DS1.11 (D4): no longer U2.25 (PC2)
- net at DS1.12 (D5): no longer U2.4 (PD2)
- net at DS1.13 (D6): no longer U2.5 (PD3)
- net at DS1.14 (D7): no longer U2.6 (PD4)
- net at DS1.15 (LED(+)): now also R6.1
- net at U2.16 (PB2): no longer DS1.4 (RS)
- net at U2.15 (PB1): no longer DS1.5 (R/W)
- net at U2.14 (PB0): no longer DS1.6 (E)
- net at U2.17 (PB3): no longer DS1.7 (D0)
- net at DS1.9 (D2): no longer U2.23 (PC0)
- net SW3: now reaches SW3.1 (A), U2.11 (PD5)
- net SW3: now also R10.2
- net SDA: now reaches U2.27 (PC4)
- net SDA: now also U1.5 (SDA), R11.2; no longer SW2.1 (A)
- net SW4: now reaches SW4.1 (A), U2.12 (PD6)
- net SW4: now also R9.2
- net at D14.4 (DOUT): now also D6.2 (DIN)
- net NEO: now reaches D2.2 (DIN), R3.2
- net SCL: now reaches U2.28 (PC5)
- net SCL: now also U1.6 (SCL), R12.2
- net at U1.1 (X1): now also Y2.2
- net at U1.2 (X2): now also Y2.1
- net at U1.3 (VBAT): now also BT1.1 (+)
- new net: D12.4 (DOUT), D13.2 (DIN)
- new net: DS1.3 (VO), RV1.2
- new net: D11.4 (DOUT), D12.2 (DIN)
- new net: D6.4 (DOUT), D7.2 (DIN)
- new net: D7.4 (DOUT), D8.2 (DIN)
- new net: C4.1, U2.9 (XTAL1/PB6), Y1.1
- new net: C5.1, U2.10 (XTAL2/PB7), Y1.2
- new net: D10.4 (DOUT), D11.2 (DIN)
- new net: D10.2 (DIN), D8.4 (DOUT)
- new net D0: DS1.7 (D0), U2.26 (PC3)
- new net E: DS1.6 (E), U2.23 (PC0)
- new net RS: DS1.4 (RS), U2.25 (PC2)
- new net RW: DS1.5 (R/W), U2.24 (PC1)
- new net SW1: R7.2, SW1.1 (A), U2.5 (PD3)
- new net SW2: R8.2, SW2.1 (A), U2.6 (PD4)
- no-connect marks 2 -> 25
Other:
- note added: "LCD"
- note added: "NEOPIXELS"
- note added: "RTC"
- note added: "SW"
- note removed: "Crystal Rectangular Schematic"
- moved on the sheet: C1, C2, C3, C4, C5, C6, C7, D1, D14, D2, D3, D4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

Commit message: LCD Edits
Parts:
- gave numbers to parts that had none: 1
Connections:
- net D4: now reaches DS1.11 (D4)
- net D4: now also U2.14 (PB0)
- net D5: now reaches DS1.12 (D5)
- net D5: now also U2.15 (PB1)
- net D6: now reaches DS1.13 (D6)
- net D6: now also U2.16 (PB2)
- net D7: now reaches DS1.14 (D7)
- net D7: now also U2.17 (PB3)
- no-connect marks 25 -> 17
Changed lines of the file:
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@@
   (no_connect (at 29.21 181.61))
   (no_connect (at 29.21 184.15))
-  (no_connect (at 29.21 194.31))
-  (no_connect (at 29.21 189.23))
-  (no_connect (at 29.21 191.77))
-  (no_connect (at 29.21 186.69))
   (no_connect (at 69.85 59.69))
-  (no_connect (at 69.85 52.07))
-  (no_connect (at 69.85 46.99))
-  (no_connect (at 69.85 49.53))
-  (no_connect (at 69.85 54.61))
   (no_connect (at 69.85 57.15))
   (no_connect (at 185.42 266.7))
@@
     (stroke (width 0) (type default) (color 0 0 0 0))
   )
-  (wire (pts (xy 24.13 168.91) (xy 24.13 170.18))
-    (stroke (width 0) (type default) (color 0 0 0 0))
-  )
   (polyline (pts (xy 129.54 54.61) (xy 129.54 60.96))
     (stroke (width 0) (type default) (color 0 0 0 0))
@@
     (stroke (width 0) (type default) (color 0 0 0 0))
   )
-  (wire (pts (xy 29.21 168.91) (xy 24.13 168.91))
-    (stroke (width 0) (type default) (color 0 0 0 0))
-  )
   (polyline (pts (xy 123.19 127) (xy 124.46 127))
     (stroke (width 0) (type default) (color 0 0 0 0))
   )
-  (wire (pts (xy 24.13 166.37) (xy 29.21 166.37))
-    (stroke (width 0) (type default) (color 0 0 0 0))
-  )
   (wire (pts (xy 54.61 25.4) (xy 54.61 39.37))
     (stroke (width 0) (type default) (color 0 0 0 0))
@@
     (stroke (width 0) (type default) (color 0 0 0 0))
   )
-  (wire (pts (xy 24.13 176.53) (xy 29.21 176.53))
-    (stroke (width 0) (type default) (color 0 0 0 0))
-  )
   (wire (pts (xy 52.07 173.99) (xy 52.07 176.53))
     (stroke (width 0) (type default) (color 0 0 0 0))
@@
     (stroke (width 0) (type default) (color 0 0 0 0))
   )
-  (wire (pts (xy 29.21 162.56) (xy 29.21 163.83))
-    (stroke (width 0) (type default) (color 0 0 0 0))
-  )
   (wire (pts (xy 22.86 52.07) (xy 22.86 46.99))
     (stroke (width 0) (type default) (color 0 0 0 0))
@@
     (stroke (width 0) (type default) (color 0 0 0 0))
   )
-  (wire (pts (xy 24.13 162.56) (xy 29.21 162.56))
-    (stroke (width 0) (type default) (color 0 0 0 0))
-  )
   (polyline (pts (xy 16.51 222.25) (xy 16.51 279.4))
     (stroke (width 0) (type default) (color 0 0 0 0))
@@
     )
   )
+  (global_label "D4" (shape input) (at 29.21 186.69 180) (fields_autoplaced)
+    (effects (font (size 1.27 1.27)) (justify right))
+    (property "Intersheet References" "${INTERSHEET_REFS}" (id 0) (at 24.3174 186.6106 0)
+      (effects (font (size 1.27 1.27)) (justify right) hide)
+    )
+  )
   (global_label "SW3" (shape input) (at 73.66 107.95 0) (fields_autoplaced)
     (effects (font (size 1.27 1.27)) (justify left))
@@
     )
   )
-  (global_label "D0" (shape input) (at 24.13 176.53 180) (fields_autoplaced)
+  (global_label "D0" (shape input) (at 29.21 176.53 180) (fields_autoplaced)
     (effects (font (size 1.27 1.27)) (justify right))
-    (property "Intersheet References" "${INTERSHEET_REFS}" (id 0) (at 19.2374 176.4506 0)
+    (property "Intersheet References" "${INTERSHEET_REFS}" (id 0) (at 24.3174 176.4506 0)
       (effects (font (size 1.27 1.27)) (justify right) hide)
     )
@@
     )
   )
+  (global_label "D4" (shape input) (at 69.85 46.99 0) (fields_autoplaced)
+    (effects (font (size 1.27 1.27)) (justify left))
+    (property "Intersheet References" "${INTERSHEET_REFS}" (id 0) (at 74.7426 47.0694 0)
+      (effects (font (size 1.27 1.27)) (justify left) hide)
+    )
+  )
   (global_label "SW4" (shape input) (at 82.55 207.01 180) (fields_autoplaced)
     (effects (font (size 1.27 1.27)) (justify right))
@@
     )
   )
-  (global_label "E" (shape input) (at 24.13 162.56 180) (fields_autoplaced)
+  (global_label "E" (shape input) (at 29.21 163.83 180) (fields_autoplaced)
+    (effects (font (size 1.27 1.27)) (justify right))
+    (property "Intersheet References" "${INTERSHEET_REFS}" (id 0) (at 25.6479 163.9094 0)
+      (effects (font (size 1.27 1.27)) (justify right) hide)
+    )
+  )
+  (global_label "D5" (shape input) (at 69.85 49.53 0) (fields_autoplaced)
+    (effects (font (size 1.27 1.27)) (justify left))
+    (property "Intersheet References" "${INTERSHEET_REFS}" (id 0) (at 74.7426 49.4506 0)
+      (effects (font (size 1.27 1.27)) (justify left) hide)
+    )
+  )
+  (global_label "D5" (shape input) (at 29.21 189.23 180) (fields_autoplaced)
     (effects (font (size 1.27 1.27)) (justify right))
-    (property "Intersheet References" "${INTERSHEET_REFS}" (id 0) (at 20.5679 162.6394 0)
+    (property "Intersheet References" "${INTERSHEET_REFS}" (id 0) (at 24.3174 189.1506 0)
       (effects (font (size 1.27 1.27)) (justify right) hide)
     )
@@
     )
   )
+  (global_label "D7" (shape input) (at 29.21 194.31 180) (fields_autoplaced)
+    (effects (font (size 1.27 1.27)) (justify right))
+    (property "Intersheet References" "${INTERSHEET_REFS}" (id 0) (at 24.3174 194.2306 0)
+      (effects (font (size 1.27 1.27)) (justify right) hide)
+    )
+  )
   (global_label "SW1" (shape input) (at 73.66 99.06 0) (fields_autoplaced)
     (effects (font (size 1.27 1.27)) (justify left))
@@
     )
   )
-  (global_label "RS" (shape input) (at 24.13 170.18 180) (fields_autoplaced)
+  (global_label "RS" (shape input) (at 29.21 168.91 180) (fields_autoplaced)
+    (effects (font (size 1.27 1.27)) (justify right))
+    (property "Intersheet References" "${INTERSHEET_REFS}" (id 0) (at 24.3174 168.8306 0)
+      (effects (font (size 1.27 1.27)) (justify right) hide)
+    )
+  )
+  (global_label "D6" (shape input) (at 29.21 191.77 180) (fields_autoplaced)
     (effects (font (size 1.27 1.27)) (justify right))
-    (property "Intersheet References" "${INTERSHEET_REFS}" (id 0) (at 19.2374 170.1006 0)
+    (property "Intersheet References" "${INTERSHEET_REFS}" (id 0) (at 24.3174 191.6906 0)
       (effects (font (size 1.27 1.27)) (justify right) hide)
     )
@@
     )
   )
+  (global_label "D6" (shape input) (at 69.85 52.07 0) (fields_autoplaced)
+    (effects (font (size 1.27 1.27)) (justify left))
+    (property "Intersheet References" "${INTERSHEET_REFS}" (id 0) (at 74.7426 51.9906 0)
+      (effects (font (size 1.27 1.27)) (justify left) hide)
+    )
+  )
   (global_label "RW" (shape input) (at 73.66 71.12 0) (fields_autoplaced)
     (effects (font (size 1.27 1.27)) (justify left))
@@
     )
   )
-  (global_label "RW" (shape input) (at 24.13 166.37 180) (fields_autoplaced)
+  (global_label "RW" (shape input) (at 29.21 166.37 180) (fields_autoplaced)
     (effects (font (size 1.27 1.27)) (justify right))
-    (property "Intersheet References" "${INTERSHEET_REFS}" (id 0) (at 18.9955 166.2906 0)
+    (property "Intersheet References" "${INTERSHEET_REFS}" (id 0) (at 24.0755 166.2906 0)
       (effects (font (size 1.27 1.27)) (justify right) hide)
     )
   )
+  (global_label "D7" (shape input) (at 69.85 54.61 0) (fields_autoplaced)
+    (effects (font (size 1.27 1.27)) (justify left))
+    (property "Intersheet References" "${INTERSHEET_REFS}" (id 0) (at 74.7426 54.5306 0)
+      (effects (font (size 1.27 1.27)) (justify left) hide)
+    )
+  )
   (symbol (lib_id "HPS:GND") (at 96.52 264.16 0) (unit 1)
     (in_bom yes) (on_board yes) (fields_autoplaced)
@@
   (symbol (lib_id "HPS:L7805") (at 127 259.08 0) (unit 1)
     (in_bom yes) (on_board yes) (fields_autoplaced)
-    (property "Reference" "U?" (id 0) (at 127 251.46 0))
+    (property "Reference" "U3" (id 0) (at 127 251.46 0))
     (property "Value" "L7805" (id 1) (at 127 254 0))
     (property "Footprint" "" (id 2) (at 127.635 262.89 0)
@@
     )
     (path "/8d8eb902-eb18-4cd8-b599-b62234c13840"
-      (reference "U?") (unit 1) (value "L7805") (footprint "")
+      (reference "U3") (unit 1) (value "L7805") (footprint "")
     )
     (path "/60c49968-9a6d-4fe7-8d50-396681c14974"

Commit message: Week 5
Other:
- note added: "Crystal Liang: Binary Clock"
- note added: "July 2022"
- moved on the sheet: R3
