File: HPS-Rect-Clock/HPS-Rect-Clock.kicad_sch (KiCad schematic)
At the start: 48 parts, among them J1 Conn_01x06, J2 PJ-102AH, SW1 Omron_B3F_SPST, SW2 Omron_B3F_SPST, SW3 Omron_B3F_SPST, SW4 Omron_B3F_SPST, SW5 Omron_B3F_SPST, U1 DS1307_DIP-8, U2 ATmega328-PU, U3 L7805, Y1 Crystal_16MHz, Y2 Crystal_32768Hz

Commit message: Week 5
Parts:
- R4, R5: value R_0805_4.7K -> R_0805_47
Connections:
- net SCL: now also U2.27 (PC4); no longer U2.28 (PC5)
- net SDA: now also U2.26 (PC3); no longer U2.27 (PC4)
- net D0: no longer names the net of DS1.7 (D0)
- net D0: no longer U2.26 (PC3)
- no-connect marks 17 -> 19
Changed lines of the file:
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@@
   (no_connect (at 69.85 57.15))
   (no_connect (at 185.42 266.7))
+  (no_connect (at 69.85 82.55))
   (no_connect (at 194.31 190.5))
+  (no_connect (at 29.21 176.53))
   (no_connect (at 274.32 110.49))
   (no_connect (at 85.09 259.08))
@@
     )
   )
-  (global_label "D0" (shape input) (at 69.85 77.47 0) (fields_autoplaced)
-    (effects (font (size 1.27 1.27)) (justify left))
-    (property "Intersheet References" "${INTERSHEET_REFS}" (id 0) (at 74.7426 77.3906 0)
-      (effects (font (size 1.27 1.27)) (justify left) hide)
-    )
-  )
   (global_label "TXD" (shape input) (at 69.85 92.71 0) (fields_autoplaced)
     (effects (font (size 1.27 1.27)) (justify left))
@@
     )
   )
-  (global_label "D0" (shape input) (at 29.21 176.53 180) (fields_autoplaced)
-    (effects (font (size 1.27 1.27)) (justify right))
-    (property "Intersheet References" "${INTERSHEET_REFS}" (id 0) (at 24.3174 176.4506 0)
-      (effects (font (size 1.27 1.27)) (justify right) hide)
-    )
-  )
   (global_label "LED_SCK" (shape input) (at 69.85 95.25 0) (fields_autoplaced)
     (effects (font (size 1.27 1.27)) (justify left))
@@
     )
   )
-  (global_label "SCL" (shape input) (at 69.85 82.55 0) (fields_autoplaced)
+  (global_label "SCL" (shape input) (at 69.85 80.01 0) (fields_autoplaced)
     (effects (font (size 1.27 1.27)) (justify left))
-    (property "Intersheet References" "${INTERSHEET_REFS}" (id 0) (at 75.7707 82.4706 0)
+    (property "Intersheet References" "${INTERSHEET_REFS}" (id 0) (at 75.7707 79.9306 0)
       (effects (font (size 1.27 1.27)) (justify left) hide)
     )
@@
     )
   )
-  (global_label "SDA" (shape input) (at 69.85 80.01 0) (fields_autoplaced)
+  (global_label "SDA" (shape input) (at 69.85 77.47 0) (fields_autoplaced)
     (effects (font (size 1.27 1.27)) (justify left))
-    (property "Intersheet References" "${INTERSHEET_REFS}" (id 0) (at 75.8312 79.9306 0)
+    (property "Intersheet References" "${INTERSHEET_REFS}" (id 0) (at 75.8312 77.3906 0)
       (effects (font (size 1.27 1.27)) (justify left) hide)
     )
@@
     (in_bom yes) (on_board yes) (fields_autoplaced)
     (property "Reference" "R4" (id 0) (at 207.01 255.27 90))
-    (property "Value" "R_0805_4.7K" (id 1) (at 207.01 257.81 90))
+    (property "Value" "R_0805_47" (id 1) (at 207.01 257.81 90))
     (property "Footprint" "footprints:R_0805_2012Metric" (id 2) (at 224.79 261.62 0)
       (effects (font (size 1.27 1.27)) hide)
@@
     (in_bom yes) (on_board yes)
     (property "Reference" "R5" (id 0) (at 207.01 269.24 90))
-    (property "Value" "R_0805_4.7K" (id 1) (at 207.01 271.78 90))
+    (property "Value" "R_0805_47" (id 1) (at 207.01 271.78 90))
     (property "Footprint" "footprints:R_0805_2012Metric" (id 2) (at 224.79 265.43 0)
       (effects (font (size 1.27 1.27)) hide)
@@
     )
     (path "/485ea5c9-b1c0-46a9-93d7-61e56150a288"
-      (reference "R4") (unit 1) (value "R_0805_4.7K") (footprint "footprints:R_0805_2012Metric")
+      (reference "R4") (unit 1) (value "R_0805_47") (footprint "footprints:R_0805_2012Metric")
     )
     (path "/c20b30ae-8c37-46f6-a56f-e5e40abbe2c8"
-      (reference "R5") (unit 1) (value "R_0805_4.7K") (footprint "footprints:R_0805_2012Metric")
+      (reference "R5") (unit 1) (value "R_0805_47") (footprint "footprints:R_0805_2012Metric")
     )
     (path "/acc43b90-8a1e-429e-9b04-6541c6d1a9b5"

Commit message: Week 6: Pre route
Parts:
- removed J2: PJ-102AH, footprints:PJ-102AH, symbol HPS:PJ-102AH
- added H1, H2, H3, H4: MountingHole, footprints:MountingHole_3.2mm_M3, symbol HPS:MountingHole
- added J2: Power_inlet_vertical, footprints:Wurth-694106402002, symbol HPS:Power_inlet_vertical
- U3: footprint (none) -> footprints:TO-252-2; Digikey PN (none) -> 497-7255-1-ND; MFG (none) -> STMicroelectronics; MPN (none) -> L7805CDT-TR
Connections:
- net D5: now also U2.16 (PB2); no longer U2.15 (PB1)
- net D6: now also U2.15 (PB1); no longer U2.16 (PB2)
- net GND: now also SW1.4 (B), SW2.4 (B), SW3.4 (B), SW4.4 (B), J2.2 (OUT)
- net SW1: now also SW1.2 (A)
- net SW2: now also SW2.2 (A)
- net SW3: now also SW3.2 (A)
- net SW4: now also SW4.2 (A)
- net at C6.2, U3.1 (IN): now also J2.1 (POLE)
- no-connect marks 19 -> 11
Other:
- note added: "Mechanical"
- moved on the sheet: R6

Commit message: PCB Placement Done
Connections:
- net D4: now also U2.17 (PB3); no longer U2.14 (PB0)
- net D7: now also U2.14 (PB0); no longer U2.17 (PB3)
Changed lines of the file:
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@@
     )
   )
-  (global_label "D4" (shape input) (at 69.85 46.99 0) (fields_autoplaced)
+  (global_label "D4" (shape input) (at 69.85 54.61 0) (fields_autoplaced)
     (effects (font (size 1.27 1.27)) (justify left))
-    (property "Intersheet References" "${INTERSHEET_REFS}" (id 0) (at 74.7426 47.0694 0)
+    (property "Intersheet References" "${INTERSHEET_REFS}" (id 0) (at 74.7426 54.6894 0)
       (effects (font (size 1.27 1.27)) (justify left) hide)
     )
@@
     )
   )
-  (global_label "D7" (shape input) (at 69.85 54.61 0) (fields_autoplaced)
+  (global_label "D7" (shape input) (at 69.85 46.99 0) (fields_autoplaced)
     (effects (font (size 1.27 1.27)) (justify left))
-    (property "Intersheet References" "${INTERSHEET_REFS}" (id 0) (at 74.7426 54.5306 0)
+    (property "Intersheet References" "${INTERSHEET_REFS}" (id 0) (at 74.7426 46.9106 0)
       (effects (font (size 1.27 1.27)) (justify left) hide)
     )

Commit message: Pre Gerber Edits
Parts:
- added J3: Conn_02x03_Odd_Even, footprints:PinHeader_2x03_P2.54mm_Vertical, symbol HPS:Conn_02x03_Odd_Even
- added TP1, TP3, TP4, TP5, TP6: TestPoint, footprints:TestPoint_THTPad_D2.0mm_Drill1.0mm, symbol HPS:TestPoint
Connections:
- net D4: now also U2.28 (PC5); no longer U2.17 (PB3)
- net GND: now also J3.6 (Pin_6)
- net NEO: now also TP1.1
- net RESET: now also J3.5 (Pin_5)
- net SW1: now also TP5.1
- net SW2: now also TP6.1
- net SW3: now also TP3.1
- net SW4: now also TP4.1
- net VCC: now also J3.2 (Pin_2)
- net MISO: now reaches U2.18 (PB4)
- net MISO: now also J3.1 (Pin_1)
- net ICSP_SCK: now reaches U2.19 (PB5)
- net ICSP_SCK: now also J3.3 (Pin_3)
- new net MOSI: J3.4 (Pin_4), U2.17 (PB3)
- no-connect marks 11 -> 8
Other:
- note added: "ICSP"
- moved on the sheet: BT1, R11, R12, U1, Y2
