File: HPS-Rect-Clock/HPS-Rect-Clock.kicad_sch (KiCad schematic)
At the start: 58 parts, among them J1 Conn_01x06, J2 Power_inlet_vertical, J3 Conn_02x03_Odd_Even, SW1 Omron_B3F_SPST, SW2 Omron_B3F_SPST, SW3 Omron_B3F_SPST, SW4 Omron_B3F_SPST, SW5 Omron_B3F_SPST, U1 DS1307_DIP-8, U2 ATmega328-PU, U3 L7805, Y1 Crystal_16MHz, Y2 Crystal_32768Hz

Commit message: Gerber out all done
Parts:
- added C10, C11, C12, C13, C14, C15, C16, C17, C18, C19, C20, C8, C9: C_0805_0.1uf, footprints:C_0805_2012Metric, symbol HPS:C_0805_0.1uf
- C7: value C_0805_0.11uf -> C_0805_0.1uf
Connections:
- net ICSP_SCK is gone; now on net LED_SCK: J3.3 (Pin_3), U2.19 (SCK/PB5)
- net GND: now also C10.1, C11.1, C12.1, C13.1, C14.1, C15.1, C16.1, C17.1, C18.1, C19.1, C20.1, C8.1, C9.1
- net VCC: now also C10.2, C11.2, C12.2, C13.2, C14.2, C15.2, C16.2, C17.2, C18.2, C19.2, C20.2, C8.2, C9.2
Other:
- note added: "NEOPIXEL CAPACITORS"
- moved on the sheet: D14, D2, D3, D4, D5, D9, H1, H2, H3, H4, R11, R12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
