File: HPS-Rect-Clock/HPS-Rect-Clock.kicad_pcb (KiCad board)
At the start: 2 copper layers, 140 x 90 mm, 4 parts

Commit message: Week 5
Parts:
- added BT1: Battery_Cell, footprints:BatteryHolder_Keystone_106_1x20mm, F.Cu at (143.3, 71.1)
- added C1: C_0805_0.1uf, footprints:C_0805_2012Metric, F.Cu at (139.7, 127.0)
- added C2: C_0805_0.1uf, footprints:C_0805_2012Metric, F.Cu at (91.4, 94.4)
- added C3: C_0805_0.1uf, footprints:C_0805_2012Metric, F.Cu at (152.7, 98.3)
- added C4: C_0805_22pf, footprints:C_0805_2012Metric, F.Cu at (87.0, 97.3)
- added C5: C_0805_22pf, footprints:C_0805_2012Metric, F.Cu at (137.7, 86.1)
- added C6: C_0805_1uf, footprints:C_0805_2012Metric, F.Cu at (148.3, 98.3)
- added C7: C_0805_0.11uf, footprints:C_0805_2012Metric, F.Cu at (148.3, 101.2)
- added D1: LED_0805, footprints:LED_0805_2012Metric, F.Cu at (100.5, 127.5)
- added D10: NEOPIXEL_SMT, footprints:LED_SK6812_PLCC4_5.0x5.0mm_P3.2mm, F.Cu at (89.0, 86.7)
- added D11: NEOPIXEL_SMT, footprints:LED_SK6812_PLCC4_5.0x5.0mm_P3.2mm, F.Cu at (122.9, 109.6)
- added D12: NEOPIXEL_SMT, footprints:LED_SK6812_PLCC4_5.0x5.0mm_P3.2mm, F.Cu at (120.0, 103.0)
- added D13: NEOPIXEL_SMT, footprints:LED_SK6812_PLCC4_5.0x5.0mm_P3.2mm, F.Cu at (134.0, 95.1)
- added D14: NEOPIXEL_SMT, footprints:LED_SK6812_PLCC4_5.0x5.0mm_P3.2mm, F.Cu at (149.9, 124.5)
- added D2: NEOPIXEL_SMT, footprints:LED_SK6812_PLCC4_5.0x5.0mm_P3.2mm, F.Cu at (139.7, 81.3)
- added D3: NEOPIXEL_SMT, footprints:LED_SK6812_PLCC4_5.0x5.0mm_P3.2mm, F.Cu at (136.8, 101.7)
- added D4: NEOPIXEL_SMT, footprints:LED_SK6812_PLCC4_5.0x5.0mm_P3.2mm, F.Cu at (111.5, 103.0)
- added D5: NEOPIXEL_SMT, footprints:LED_SK6812_PLCC4_5.0x5.0mm_P3.2mm, F.Cu at (119.5, 124.6)
- added D6: NEOPIXEL_SMT, footprints:LED_SK6812_PLCC4_5.0x5.0mm_P3.2mm, F.Cu at (122.9, 116.2)
- added D7: NEOPIXEL_SMT, footprints:LED_SK6812_PLCC4_5.0x5.0mm_P3.2mm, F.Cu at (128.4, 103.0)
- added D8: NEOPIXEL_SMT, footprints:LED_SK6812_PLCC4_5.0x5.0mm_P3.2mm, F.Cu at (97.5, 86.7)
- added D9: NEOPIXEL_SMT, footprints:LED_SK6812_PLCC4_5.0x5.0mm_P3.2mm, F.Cu at (131.3, 109.6)
- added DS1: TC1602A-01T, footprints:TC1602A-01T, F.Cu at (175.1, 131.1)
- added J1: Conn_01x06, footprints:PinHeader_1x06_P2.54mm_Vertical, F.Cu at (104.1, 64.8)
- added J2: PJ-102AH, footprints:PJ-102AH, F.Cu at (132.1, 71.6)
- added R1: R_0805_2.2K, footprints:R_0805_2012Metric, F.Cu at (93.3, 70.3)
- added R10: R_0805_10K, footprints:R_0805_2012Metric, F.Cu at (87.0, 94.4)
- added R11: R_0805_4.7K, footprints:R_0805_2012Metric, F.Cu at (152.7, 101.2)
- added R12: R_0805_4.7K, footprints:R_0805_2012Metric, F.Cu at (151.1, 104.2)
- added R2: R_0805_10K, footprints:R_0805_2012Metric, F.Cu at (125.9, 126.0)
- added R3: R_0805_47, footprints:R_0805_2012Metric, F.Cu at (149.9, 114.3)
- added R4: R_0805_47, footprints:R_0805_2012Metric, F.Cu at (88.9, 76.2)
- added R5: R_0805_47, footprints:R_0805_2012Metric, F.Cu at (88.9, 73.2)
- added R6: R_0805_47, footprints:R_0805_2012Metric, F.Cu at (91.4, 91.4)
- added R7: R_0805_10K, footprints:R_0805_2012Metric, F.Cu at (137.7, 106.5)
- added R8: R_0805_10K, footprints:R_0805_2012Metric, F.Cu at (87.0, 91.4)
- added R9: R_0805_10K, footprints:R_0805_2012Metric, F.Cu at (88.9, 70.3)
- added RV1: R_POT_10K, footprints:Potentiometer_Bourns_3386P_Vertical, F.Cu at (116.8, 71.1)
- added SW1: Omron_B3F_SPST, footprints:SW_SPST_Omron_B3FS-100xP, F.Cu at (96.5, 137.2)
- added SW2: Omron_B3F_SPST, footprints:SW_SPST_Omron_B3FS-100xP, F.Cu at (109.2, 137.2)
- added SW3: Omron_B3F_SPST, footprints:SW_SPST_Omron_B3FS-100xP, F.Cu at (121.9, 137.2)
- added SW4: Omron_B3F_SPST, footprints:SW_SPST_Omron_B3FS-100xP, F.Cu at (134.6, 137.2)
- added SW5: Omron_B3F_SPST, footprints:SW_SPST_Omron_B3FS-100xP, F.Cu at (147.3, 137.2)
- added U1: DS1307_DIP-8, footprints:DIP-8_W7.62mm, F.Cu at (158.8, 90.2)
- added U2: ATmega328-PU, footprints:DIP-28_W7.62mm, F.Cu at (158.8, 105.4)
- added Y1: Crystal_16MHz, footprints:Crystal_SMD_HC49-SD, F.Cu at (91.4, 116.8)
- added Y2: Crystal_32768Hz, footprints:Crystal_SMD_2Pin_3.2x1.5mm, F.Cu at (100.8, 124.2)

Commit message: Week 6: Pre route
Parts:
- added U3: L7805, footprints:TO-252-2, F.Cu at (172.3, 135.6)
- BT1: moved to B.Cu
- J2: value PJ-102AH -> Power_inlet_vertical; footprint footprints:PJ-102AH -> footprints:Wurth-694106402002; moved to B.Cu
- moved SW1 149.5 mm to (236.2, 83.8)
- moved SW2 134.3 mm to (238.8, 101.6)
- moved SW3 122.6 mm to (243.8, 124.5)
- moved Y2 103.9 mm to (203.2, 106.7), turned to 90 degrees
- moved C1 103.7 mm to (50.8, 73.7)
- moved C6 103.7 mm to (59.4, 45.0)
- moved D11 103.7 mm to (34.0, 56.3)
- moved D12 103.7 mm to (31.1, 49.6)
- moved D13 103.7 mm to (45.1, 41.8)
- moved D5 103.7 mm to (30.6, 71.3)
- moved D6 103.7 mm to (34.0, 62.9)
- moved D7 103.7 mm to (39.5, 49.6)
- moved D9 103.7 mm to (42.4, 56.3)
- moved R2 103.7 mm to (37.0, 72.7)
- moved R3 103.7 mm to (61.0, 61.0)
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Connections:
- SW1 pad 2: unconnected-(SW1-Pad2) -> SW1
- SW1 pad 4: unconnected-(SW1-Pad4) -> GND
- SW2 pad 2: unconnected-(SW2-Pad2) -> SW2
- SW2 pad 4: unconnected-(SW2-Pad4) -> GND
- SW3 pad 2: unconnected-(SW3-Pad2) -> SW3
- SW3 pad 4: unconnected-(SW3-Pad4) -> GND
- SW4 pad 2: unconnected-(SW4-Pad2) -> SW4
- SW4 pad 4: unconnected-(SW4-Pad4) -> GND
Routing:
- added copper zone on B.Cu, net GND
- added copper zone on F.Cu, net VCC

Commit message: PCB Placement Done
Parts:
- moved R2 183.1 mm to (215.9, 111.8), turned to 90 degrees
- moved R7 170.9 mm to (215.9, 96.5), turned to 90 degrees
- moved R6 149.9 mm to (141.7, 61.1), turned to 180 degrees
- moved R1 146.8 mm to (200.7, 106.7), turned to 90 degrees
- moved D4 145.4 mm to (147.3, 124.5)
- moved C7 144.3 mm to (170.2, 140.3)
- moved C6 139.8 mm to (170.2, 130.1)
- moved C1 136.5 mm to (185.4, 96.5), turned to 90 degrees
- moved R10 131.9 mm to (215.9, 76.2), turned to 90 degrees
- moved D5 131.6 mm to (147.3, 132.1)
- moved R8 129.2 mm to (215.9, 91.4), turned to 90 degrees
- moved R3 126.5 mm to (185.4, 83.8), turned to 90 degrees
- moved R9 121.9 mm to (215.9, 68.6), turned to -90 degrees
- moved D3 120.7 mm to (147.3, 116.8)
- moved D9 117.4 mm to (132.1, 132.1)
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Connections:
- U2 pad 14: D4 -> D7
- U2 pad 15: D5 -> D6
- U2 pad 16: D6 -> D5
- U2 pad 17: D7 -> D4

Commit message: PCB routing done p2
Parts:
- moved C4 24.1 mm to (198.1, 86.4)
- moved Y1 19.2 mm to (205.7, 83.0), turned to 90 degrees
- moved R9 18.5 mm to (198.1, 63.5)
- moved SW4 18.5 mm to (190.5, 63.5)
- moved C2 14.4 mm to (182.9, 71.1), turned to 90 degrees
- moved SW3 10.5 mm to (205.7, 68.6)
- moved R10 8.03 mm to (213.4, 68.6)
- moved SW2 7.62 mm to (208.3, 96.5)
- moved C5 5.68 mm to (198.1, 81.3)
- moved R7 5.08 mm to (215.9, 101.6)
- moved R8 5.08 mm to (215.9, 96.5)
- moved SW1 5.08 mm to (208.3, 104.1)
- moved D1 3.59 mm to (198.1, 104.1)
- moved C1 3.59 mm to (182.9, 94.0)
- moved R1 3.59 mm to (198.1, 109.2)
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Changed lines of the file:
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@@
   (net 57 "unconnected-(U2-Pad28)")
   (footprint "footprints:R_0805_2012Metric" (layer "F.Cu")
-    (at 215.9 111.76 90)
+    (at 215.9 114.3 90)
     (descr "Resistor SMD 0805 (2012 Metric), square (rectangular) end terminal, IPC_7351 nominal, (Body size source: http://www.tortai-tech.com/upload/download/2011102023233369053.pdf), generated with kicad-footprint-generator")
     (tags "resistor")
@@
   )
   (footprint "footprints:SW_SPST_Omron_B3FS-100xP" (layer "F.Cu")
-    (at 208.28 99.06)
+    (at 208.28 104.14)
     (descr "Surface Mount Tactile Switch for High-Density Mounting, 3.1mm height, https://omronfs.omron.com/en_US/ecb/products/pdf/en-b3fs.pdf")
     (tags "Tactile Switch")
@@
   )
   (footprint "footprints:R_0805_2012Metric" (layer "F.Cu")
-    (at 185.42 83.82 90)
+    (at 182.88 81.28 90)
     (descr "Resistor SMD 0805 (2012 Metric), square (rectangular) end terminal, IPC_7351 nominal, (Body size source: http://www.tortai-tech.com/upload/download/2011102023233369053.pdf), generated with kicad-footprint-generator")
     (tags "resistor")
@@
   )
   (footprint "footprints:SW_SPST_Omron_B3FS-100xP" (layer "F.Cu")
-    (at 208.28 78.74)
+    (at 205.74 68.58)
     (descr "Surface Mount Tactile Switch for High-Density Mounting, 3.1mm height, https://omronfs.omron.com/en_US/ecb/products/pdf/en-b3fs.pdf")
     (tags "Tactile Switch")
@@
   )
   (footprint "footprints:SW_SPST_Omron_B3FS-100xP" (layer "F.Cu")
-    (at 208.28 88.9 180)
+    (at 208.28 96.52 180)
     (descr "Surface Mount Tactile Switch for High-Density Mounting, 3.1mm height, https://omronfs.omron.com/en_US/ecb/products/pdf/en-b3fs.pdf")
     (tags "Tactile Switch")
@@
   )
   (footprint "footprints:R_0805_2012Metric" (layer "F.Cu")
-    (at 215.9 68.58 -90)
+    (at 198.12 63.5 -90)
     (descr "Resistor SMD 0805 (2012 Metric), square (rectangular) end terminal, IPC_7351 nominal, (Body size source: http://www.tortai-tech.com/upload/download/2011102023233369053.pdf), generated with kicad-footprint-generator")
     (tags "resistor")
@@
   )
   (footprint "footprints:C_0805_2012Metric" (layer "F.Cu")
-    (at 182.88 67.73 90)
+    (at 198.12 86.36 90)
     (descr "Capacitor SMD 0805 (2012 Metric), square (rectangular) end terminal, IPC_7351 nominal, (Body size source: http://www.tortai-tech.com/upload/download/2011102023233369053.pdf), generated with kicad-footprint-generator")
     (tags "capacitor")
@@
   )
   (footprint "footprints:R_0805_2012Metric" (layer "F.Cu")
-    (at 200.66 106.68 90)
+    (at 198.12 109.22 90)
     (descr "Resistor SMD 0805 (2012 Metric), square (rectangular) end terminal, IPC_7351 nominal, (Body size source: http://www.tortai-tech.com/upload/download/2011102023233369053.pdf), generated with kicad-footprint-generator")
     (tags "resistor")
@@
   )
   (footprint "footprints:R_0805_2012Metric" (layer "F.Cu")
-    (at 215.9 91.44 90)
+    (at 215.9 96.52 90)
     (descr "Resistor SMD 0805 (2012 Metric), square (rectangular) end terminal, IPC_7351 nominal, (Body size source: http://www.tortai-tech.com/upload/download/2011102023233369053.pdf), generated with kicad-footprint-generator")
     (tags "resistor")
@@
   )
   (footprint "footprints:DIP-28_W7.62mm" (layer "F.Cu")
-    (at 196.84 107.94 180)
+    (at 194.3 105.4 180)
     (descr "28-lead though-hole mounted DIP package, row spacing 7.62 mm (300 mils)")
     (tags "THT DIP DIL PDIP 2.54mm 7.62mm 300mil")
@@
   )
   (footprint "footprints:SW_SPST_Omron_B3FS-100xP" (layer "F.Cu")
-    (at 208.28 109.22)
+    (at 208.28 111.76)
     (descr "Surface Mount Tactile Switch for High-Density Mounting, 3.1mm height, https://omronfs.omron.com/en_US/ecb/products/pdf/en-b3fs.pdf")
     (tags "Tactile Switch")
@@
   )
   (footprint "footprints:R_0805_2012Metric" (layer "F.Cu")
-    (at 215.9 76.2 90)
+    (at 213.36 68.58 90)
     (descr "Resistor SMD 0805 (2012 Metric), square (rectangular) end terminal, IPC_7351 nominal, (Body size source: http://www.tortai-tech.com/upload/download/2011102023233369053.pdf), generated with kicad-footprint-generator")
     (tags "resistor")
@@
   )
   (footprint "footprints:Crystal_SMD_HC49-SD" (layer "F.Cu")
-    (at 193.04 68.58)
+    (at 205.74 82.99 90)
     (descr "SMD Crystal HC-49-SD http://cdn-reichelt.de/documents/datenblatt/B400/xxx-HC49-SMD.pdf, 11.4x4.7mm^2 package")
     (tags "SMD SMT crystal")
@@
     (property "Sheetname" "")
     (attr smd)
-    (fp_text reference "Y1" (at 0 -3.55) (layer "F.SilkS")
-      (effects (font (size 1 1) (thickness 0.15)))
-    )
-    (fp_text value "Crystal_16MHz" (at 0 3.55) (layer "F.Fab")
-      (effects (font (size 1 1) (thickness 0.15)))
-    )
-    (fp_text user "${REFERENCE}" (at 0 2.115) (layer "F.Fab")
+    (fp_text reference "Y1" (at 0 -3.55 90) (layer "F.SilkS")
+      (effects (font (size 1 1) (thickness 0.15)))
+    )
+    (fp_text value "Crystal_16MHz" (at 0 3.55 90) (layer "F.Fab")
+      (effects (font (size 1 1) (thickness 0.15)))
+    )
+    (fp_text user "${REFERENCE}" (at 0 2.115 90) (layer "F.Fab")
       (effects (font (size 1 1) (thickness 0.15)))
     )
@@
     (fp_arc (start -3.015 2.115) (mid -5.13 0) (end -3.015 -2.115) (layer "F.Fab") (width 0.1))
     (fp_arc (start 3.015 -2.115) (mid 5.13 0) (end 3.015 2.115) (layer "F.Fab") (width 0.1))
-    (pad "1" smd rect locked (at -4.25 0) (size 4.5 2) (layers "F.Cu" "F.Paste" "F.Mask")
+    (pad "1" smd rect locked (at -4.25 0 90) (size 4.5 2) (layers "F.Cu" "F.Paste" "F.Mask")
       (net 7 "Net-(C4-Pad1)") (pinfunction "1") (pintype "passive"))
-    (pad "2" smd rect locked (at 4.25 0) (size 4.5 2) (layers "F.Cu" "F.Paste" "F.Mask")
+    (pad "2" smd rect locked (at 4.25 0 90) (size 4.5 2) (layers "F.Cu" "F.Paste" "F.Mask")
       (net 8 "Net-(C5-Pad1)") (pinfunction "2") (pintype "passive"))
     (model "${HPS3DMOD}/Crystal_SMD_HC49-SD.wrl"
@@
   )
   (footprint "footprints:SW_SPST_Omron_B3FS-100xP" (layer "F.Cu")
-    (at 208.28 68.58 180)
+    (at 190.5 63.5 180)
     (descr "Surface Mount Tactile Switch for High-Density Mounting, 3.1mm height, https://omronfs.omron.com/en_US/ecb/products/pdf/en-b3fs.pdf")
     (tags "Tactile Switch")
@@
   )
   (footprint "footprints:LED_0805_2012Metric" (layer "F.Cu")
-    (at 200.66 101.6 90)
+    (at 198.12 104.14 90)
     (descr "LED SMD 0805 (2012 Metric), square (rectangular) end terminal, IPC_7351 nominal, (Body size source: https://docs.google.com/spreadsheets/d/1BsfQQcO9C6DZCsRaXUlFlo91Tg2WpOkGARC1WS5S8t0/edit?usp=sharing), generated with kicad-footprint-generator")
     (tags "LED")
@@
   )
   (footprint "footprints:R_0805_2012Metric" (layer "F.Cu")
-    (at 215.9 96.52 90)
+    (at 215.9 101.6 90)
     (descr "Resistor SMD 0805 (2012 Metric), square (rectangular) end terminal, IPC_7351 nominal, (Body size source: http://www.tortai-tech.com/upload/download/2011102023233369053.pdf), generated with kicad-footprint-generator")
     (tags "resistor")
@@
   )
   (footprint "footprints:C_0805_2012Metric" (layer "F.Cu")
-    (at 193.04 60.96)
+    (at 182.88 71.12 90)
     (descr "Capacitor SMD 0805 (2012 Metric), square (rectangular) end terminal, IPC_7351 nominal, (Body size source: http://www.tortai-tech.com/upload/download/2011102023233369053.pdf), generated with kicad-footprint-generator")
     (tags "capacitor")
@@
     (property "Voltage" "N/A")
     (attr smd)
-    (fp_text reference "C2" (at 0 -1.65) (layer "F.SilkS")
-      (effects (font (size 1 1) (thickness 0.15)))
-    )
-    (fp_text value "C_0805_0.1uf" (at 0 1.65) (layer "F.Fab")
-      (effects (font (size 1 1) (thickness 0.15)))
-    )
-    (fp_text user "${REFERENCE}" (at 0 0) (layer "F.Fab")
+    (fp_text reference "C2" (at 0 -1.65 90) (layer "F.SilkS")
+      (effects (font (size 1 1) (thickness 0.15)))
+    )
+    (fp_text value "C_0805_0.1uf" (at 0 1.65 90) (layer "F.Fab")
+      (effects (font (size 1 1) (thickness 0.15)))
+    )
+    (fp_text user "${REFERENCE}" (at 0 0 90) (layer "F.Fab")
       (effects (font (size 0.5 0.5) (thickness 0.08)))
     )
@@
     (fp_line (start 1 -0.6) (end 1 0.6) (layer "F.Fab") (width 0.1))
     (fp_line (start -1 0.6) (end -1 -0.6) (layer "F.Fab") (width 0.1))
-    (pad "1" smd rect locked (at -0.85 0) (size 1.15 1.4) (layers "F.Cu" "F.Paste" "F.Mask")
+    (pad "1" smd rect locked (at -0.85 0 90) (size 1.15 1.4) (layers "F.Cu" "F.Paste" "F.Mask")
       (net 4 "VCC") (pintype "passive"))
-    (pad "2" smd rect locked (at 0.85 0) (size 1.15 1.4) (layers "F.Cu" "F.Paste" "F.Mask")
+    (pad "2" smd rect locked (at 0.85 0 90) (size 1.15 1.4) (layers "F.Cu" "F.Paste" "F.Mask")
       (net 1 "GND") (pintype "passive"))
     (model "${HPS3DMOD}/C_0805_2012Metric.wrl"
@@
   )
   (footprint "footprints:C_0805_2012Metric" (layer "F.Cu")
-    (at 185.42 96.52 90)
+    (at 182.88 93.98 90)
     (descr "Capacitor SMD 0805 (2012 Metric), square (rectangular) end terminal, IPC_7351 nominal, (Body size source: http://www.tortai-tech.com/upload/download/2011102023233369053.pdf), generated with kicad-footprint-generator")
     (tags "capacitor")
@@
   )
   (footprint "footprints:C_0805_2012Metric" (layer "F.Cu")
-    (at 200.66 86.36 90)
+    (at 198.12 81.28 90)
     (descr "Capacitor SMD 0805 (2012 Metric), square (rectangular) end terminal, IPC_7351 nominal, (Body size source: http://www.tortai-tech.com/upload/download/2011102023233369053.pdf), generated with kicad-footprint-generator")
     (tags "capacitor")
@@
       (effects (font (size 1 1) (thickness 0.15)))
     )
-    (fp_text user "${REFERENCE}" (at 0 0 90) (layer "F.Fab")
+    (fp_text user "${REFERENCE}" (at 2.54 -0.6 90) (layer "F.Fab")
       (effects (font (size 0.5 0.5) (thickness 0.08)))
     )

Commit message: Starting Traces
Parts:
- moved RV1 38.7 mm to (129.5, 106.7)
- moved C7 26.5 mm to (165.1, 114.3)
- moved J2 26.5 mm to (156.5, 109.2)
- moved U3 26.5 mm to (167.6, 109.2)
- moved C6 26.5 mm to (165.1, 104.1)
- moved R12 24.3 mm to (156.1, 129.1)
- moved R11 24.3 mm to (156.1, 124.0)
- moved U1 24.3 mm to (167.6, 132.9)
- moved Y2 24.3 mm to (171.4, 131.6)
- moved J1 10.2 mm to (180.3, 113.0)
- moved R5 7.48 mm to (185.4, 109.2)
- moved R4 5.62 mm to (185.4, 114.3)
- moved C3 5.08 mm to (190.5, 116.7)
- moved D14 2.54 mm to (129.5, 124.5)
- moved D6 2.54 mm to (129.5, 116.8)
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Routing:
- net Net-(DS1-Pad3): track 0.00 -> 100.3 mm

Commit message: Moderate amount of tracing done
Parts:
- moved R6 13.7 mm to (128.7, 65.4)
- moved DS1 11.9 mm to (93.3, 69.8)
- moved C2 8.03 mm to (180.3, 63.5)
- moved R3 7.59 mm to (179.1, 87.8), turned to -90 degrees
- moved C1 6.38 mm to (183.5, 87.6), turned to -90 degrees
- moved R4 5.85 mm to (191.1, 115.6)
- moved C3 5.61 mm to (196.0, 115.6)
- moved C5 5.43 mm to (200.0, 76.2), turned to -90 degrees
- moved C4 4.96 mm to (201.3, 90.2), turned to -90 degrees
- moved C7 4.76 mm to (166.8, 118.7)
- moved D14 3.99 mm to (131.5, 127.9)
- moved J2 3.99 mm to (158.5, 112.7)
- moved R11 3.99 mm to (158.1, 127.5)
- moved U3 3.99 mm to (169.6, 112.7)
- moved U1 3.99 mm to (169.5, 136.4)
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Routing:
- net GND: track 0.00 -> 416.0 mm
- net Net-(DS1-Pad3): track 100.3 -> 50.4 mm
- net SCL: track 0.00 -> 49.3 mm
- net Net-(D6-Pad4): track 0.00 -> 19.3 mm
- net Net-(BT1-Pad1): track 0.00 -> 19.2 mm
- net SW4: track 0.00 -> 15.8 mm
- net Net-(D12-Pad4): track 0.00 -> 12.6 mm
- net Net-(C6-Pad2): track 0.00 -> 12.5 mm
- net Net-(D5-Pad4): track 0.00 -> 11.7 mm
- net Net-(D11-Pad4): track 0.00 -> 11.7 mm
- net Net-(D14-Pad2): track 0.00 -> 10.8 mm
- net Net-(D10-Pad4): track 0.00 -> 6.73 mm
- net Net-(D4-Pad4): track 0.00 -> 6.73 mm
- net Net-(D2-Pad4): track 0.00 -> 6.73 mm
- net Net-(D7-Pad4): track 0.00 -> 6.73 mm
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
Commit message: Tracing nearly done
Parts:
- moved R8 15.2 mm to (200.7, 96.1)
- moved R7 14.6 mm to (201.3, 101.4)
- moved R4 2.94 mm to (189.7, 113.0)
- moved R2 0.64 mm to (215.3, 114.3)
- moved R10 0.63 mm to (214.0, 68.6), turned to -90 degrees
- moved SW2 0.63 mm to (208.3, 95.9)
- moved SW5 0.63 mm to (208.3, 112.4)
- turned R1 to -90 degrees
Routing:
- net GND: track 416.0 -> 544.1 mm
- net RS: track 0.00 -> 97.9 mm
- net RW: track 0.00 -> 94.3 mm
- net E: track 0.00 -> 90.7 mm
- net D4: track 0.00 -> 71.7 mm
- net D7: track 0.00 -> 70.1 mm
- net D5: track 0.00 -> 68.1 mm
- net D6: track 0.00 -> 64.5 mm
- net SDA: track 4.67 -> 47.6 mm
- net RESET: track 0.00 -> 32.7 mm
- net SW3: track 0.00 -> 27.2 mm
- net SW1: track 0.00 -> 22.0 mm
- net Net-(R3-Pad1): track 0.00 -> 20.9 mm
- net SW2: track 0.00 -> 19.6 mm
- net Net-(C5-Pad1): track 0.00 -> 18.3 mm
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