File: HPS-Rect-Clock/HPS-Rect-Clock.kicad_pcb (KiCad board)
At the start: 2 copper layers, 140 x 90 mm, 58 parts, among them J1 Conn_01x06, J2 Power_inlet_vertical, J3 Conn_02x03_Odd_Even, SW1 Omron_B3F_SPST, SW2 Omron_B3F_SPST, SW3 Omron_B3F_SPST, SW4 Omron_B3F_SPST, SW5 Omron_B3F_SPST, U1 DS1307_DIP-8, U2 ATmega328-PU, U3 L7805, Y1 Crystal_16MHz, Y2 Crystal_32768Hz

Commit message: Gerber out all done
Parts:
- added C10: C_0805_0.1uf, footprints:C_0805_2012Metric, F.Cu at (110.3, 120.7)
- added C11: C_0805_0.1uf, footprints:C_0805_2012Metric, F.Cu at (140.9, 112.6)
- added C12: C_0805_0.1uf, footprints:C_0805_2012Metric, F.Cu at (140.8, 120.7)
- added C13: C_0805_0.1uf, footprints:C_0805_2012Metric, F.Cu at (125.5, 120.0)
- added C14: C_0805_0.1uf, footprints:C_0805_2012Metric, F.Cu at (110.5, 137.2)
- added C15: C_0805_0.1uf, footprints:C_0805_2012Metric, F.Cu at (94.0, 135.9)
- added C16: C_0805_0.1uf, footprints:C_0805_2012Metric, F.Cu at (94.4, 129.5)
- added C17: C_0805_0.1uf, footprints:C_0805_2012Metric, F.Cu at (124.5, 128.3)
- added C18: C_0805_0.1uf, footprints:C_0805_2012Metric, F.Cu at (125.7, 137.2)
- added C19: C_0805_0.1uf, footprints:C_0805_2012Metric, F.Cu at (141.0, 128.9)
- added C20: C_0805_0.1uf, footprints:C_0805_2012Metric, F.Cu at (110.5, 112.4)
- added C8: C_0805_0.1uf, footprints:C_0805_2012Metric, F.Cu at (110.3, 127.6)
- added C9: C_0805_0.1uf, footprints:C_0805_2012Metric, F.Cu at (140.8, 137.2)
- C7: value C_0805_0.11uf -> C_0805_0.1uf
- moved R1 33.4 mm to (179.7, 83.2), turned to 180 degrees
- moved D1 25.4 mm to (183.8, 83.2), turned to 0 degrees
Connections:
- J3 pad 3: ICSP_SCK -> LED_SCK
- U2 pad 19: ICSP_SCK -> LED_SCK
- U2 pad 4: LED_SCK -> unconnected-(U2-Pad4)
Routing:
- net ICSP_SCK: track 46.4 -> 0.00 mm, vias 1 -> 0
- net LED_SCK: track 8.48 -> 49.2 mm, vias 2 -> 1
- net GND: track 81.4 -> 119.2 mm, vias 31 -> 41
- net Net-(D12-Pad4): track 12.6 -> 9.31 mm
- net Net-(D1-Pad1): track 4.50 -> 2.35 mm
Other:
- board text added: "Binary Arc Reactor"
