File: HPS-Rect-Clock/_autosave-HPS-Rect-Clock.kicad_sch (KiCad schematic)
At the start: 53 parts, among them J1 Conn_01x06, J2 Power_inlet_vertical, SW1 Omron_B3F_SPST, SW2 Omron_B3F_SPST, SW3 Omron_B3F_SPST, SW4 Omron_B3F_SPST, SW5 Omron_B3F_SPST, U1 DS1307_DIP-8, U2 ATmega328-PU, U3 L7805, Y1 Crystal_16MHz, Y2 Crystal_32768Hz

Commit message: test points added
Parts:
- added TP2, TP3, TP4, TP5, TP6: TestPoint, footprints:TestPoint_THTPad_D2.0mm_Drill1.0mm, symbol HPS:TestPoint
Connections:
- net SW1: now also TP5.1
- net SW2: now also TP6.1
- net SW3: now also TP3.1
- net SW4: now also TP4.1
- net at C4.1, U2.9 (XTAL1/PB6), Y1.1: now also TP2.1
Changed lines of the file:
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@@
   (junction (at 96.52 172.72) (diameter 0) (color 0 0 0 0)
   )
+  (junction (at 90.1039 207.01) (diameter 0) (color 0 0 0 0)
+  )
   (junction (at 97.79 85.09) (diameter 0) (color 0 0 0 0)
   )
+  (junction (at 99.06 172.72) (diameter 0) (color 0 0 0 0)
+  )
   (junction (at 86.36 59.69) (diameter 0) (color 0 0 0 0)
   )
+  (junction (at 90.17 190.5) (diameter 0) (color 0 0 0 0)
+  )
   (junction (at 116.84 207.01) (diameter 0) (color 0 0 0 0)
   )
@@
   (junction (at 100.33 254) (diameter 0) (color 0 0 0 0)
   )
+  (junction (at 81.28 59.69) (diameter 0) (color 0 0 0 0)
+  )
   (junction (at 149.86 175.26) (diameter 0) (color 0 0 0 0)
   )
@@
   (junction (at 116.84 154.94) (diameter 0) (color 0 0 0 0)
   )
+  (junction (at 99.06 154.94) (diameter 0) (color 0 0 0 0)
+  )
   (junction (at 149.86 190.5) (diameter 0) (color 0 0 0 0)
   )
@@
     (stroke (width 0) (type default) (color 0 0 0 0))
   )
+  (wire (pts (xy 100.33 166.37) (xy 99.06 172.72))
+    (stroke (width 0) (type default) (color 0 0 0 0))
+  )
   (wire (pts (xy 233.68 85.09) (xy 237.49 85.09))
     (stroke (width 0) (type default) (color 0 0 0 0))
@@
     (stroke (width 0) (type default) (color 0 0 0 0))
   )
+  (wire (pts (xy 90.17 184.15) (xy 90.17 190.5))
+    (stroke (width 0) (type default) (color 0 0 0 0))
+  )
   (wire (pts (xy 196.85 106.68) (xy 194.31 106.68))
     (stroke (width 0) (type default) (color 0 0 0 0))
@@
     (stroke (width 0) (type default) (color 0 0 0 0))
   )
-  (wire (pts (xy 78.74 59.69) (xy 86.36 59.69))
+  (wire (pts (xy 78.74 59.69) (xy 81.28 59.69))
     (stroke (width 0) (type default) (color 0 0 0 0))
   )
@@
     (stroke (width 0) (type default) (color 0 0 0 0))
   )
-  (wire (pts (xy 82.55 207.01) (xy 97.79 207.01))
+  (wire (pts (xy 82.55 207.01) (xy 90.1039 207.01))
     (stroke (width 0) (type default) (color 0 0 0 0))
   )
@@
     (stroke (width 0) (type default) (color 0 0 0 0))
   )
+  (wire (pts (xy 90.17 201.93) (xy 90.1039 207.01))
+    (stroke (width 0) (type default) (color 0 0 0 0))
+  )
   (wire (pts (xy 116.84 207.01) (xy 116.84 209.55))
     (stroke (width 0) (type default) (color 0 0 0 0))
@@
     (stroke (width 0) (type default) (color 0 0 0 0))
   )
+  (wire (pts (xy 81.28 59.69) (xy 86.36 59.69))
+    (stroke (width 0) (type default) (color 0 0 0 0))
+  )
   (wire (pts (xy 22.86 52.07) (xy 22.86 46.99))
     (stroke (width 0) (type default) (color 0 0 0 0))
@@
     (stroke (width 0) (type default) (color 0 0 0 0))
   )
+  (wire (pts (xy 99.06 154.94) (xy 102.87 154.94))
+    (stroke (width 0) (type default) (color 0 0 0 0))
+  )
   (wire (pts (xy 165.1 175.26) (xy 149.86 175.26))
     (stroke (width 0) (type default) (color 0 0 0 0))
@@
     (stroke (width 0) (type default) (color 0 0 0 0))
   )
-  (wire (pts (xy 96.52 172.72) (xy 102.87 172.72))
+  (wire (pts (xy 96.52 172.72) (xy 99.06 172.72))
     (stroke (width 0) (type default) (color 0 0 0 0))
   )
@@
     (stroke (width 0) (type default) (color 0 0 0 0))
   )
+  (wire (pts (xy 90.17 190.5) (xy 99.06 190.5))
+    (stroke (width 0) (type default) (color 0 0 0 0))
+  )
   (wire (pts (xy 45.72 156.21) (xy 49.53 156.21))
     (stroke (width 0) (type default) (color 0 0 0 0))
@@
     (stroke (width 0) (type default) (color 0 0 0 0))
   )
+  (wire (pts (xy 90.1039 207.01) (xy 97.79 207.01))
+    (stroke (width 0) (type default) (color 0 0 0 0))
+  )
   (wire (pts (xy 276.86 106.68) (xy 274.32 106.68))
     (stroke (width 0) (type default) (color 0 0 0 0))
@@
     (stroke (width 0) (type default) (color 0 0 0 0))
   )
-  (wire (pts (xy 82.55 190.5) (xy 99.06 190.5))
+  (wire (pts (xy 82.55 190.5) (xy 90.17 190.5))
     (stroke (width 0) (type default) (color 0 0 0 0))
   )
@@
     (stroke (width 0) (type default) (color 0 0 0 0))
   )
+  (wire (pts (xy 81.28 53.34) (xy 81.28 59.69))
+    (stroke (width 0) (type default) (color 0 0 0 0))
+  )
   (wire (pts (xy 81.28 265.43) (xy 92.71 261.62))
     (stroke (width 0) (type default) (color 0 0 0 0))
@@
     (stroke (width 0) (type default) (color 0 0 0 0))
   )
-  (wire (pts (xy 93.98 154.94) (xy 102.87 154.94))
+  (wire (pts (xy 93.98 154.94) (xy 99.06 154.94))
     (stroke (width 0) (type default) (color 0 0 0 0))
   )
@@
     (stroke (width 0) (type default) (color 0 0 0 0))
   )
+  (wire (pts (xy 99.06 172.72) (xy 102.87 172.72))
+    (stroke (width 0) (type default) (color 0 0 0 0))
+  )
   (polyline (pts (xy 16.51 16.51) (xy 16.51 127))
     (stroke (width 0) (type default) (color 0 0 0 0))
@@
     (stroke (width 0) (type default) (color 0 0 0 0))
   )
+  (wire (pts (xy 99.06 147.32) (xy 99.06 154.94))
+    (stroke (width 0) (type default) (color 0 0 0 0))
+  )
   (wire (pts (xy 233.68 110.49) (xy 237.49 110.49))
     (stroke (width 0) (type default) (color 0 0 0 0))
@@
     (pin "2")
   )
+  (symbol (lib_id "HPS:TestPoint") (at 90.17 184.15 0) (unit 1)
+    (in_bom yes) (on_board yes) (fields_autoplaced)
+    (property "Reference" "TP3" (id 0) (at 92.71 179.5779 0)
+      (effects (font (size 1.27 1.27)) (justify left))
+    )
+    (property "Value" "TestPoint" (id 1) (at 92.71 182.1179 0)
+      (effects (font (size 1.27 1.27)) (justify left))
+    )
+    (property "Footprint" "footprints:TestPoint_THTPad_D2.0mm_Drill1.0mm" (id 2) (at 95.25 184.15 0)
+      (effects (font (size 1.27 1.27)) hide)
+    )
+    (property "Datasheet" "~" (id 3) (at 95.25 184.15 0)
+      (effects (font (size 1.27 1.27)) hide)
+    )
+    (pin "1")
+  )
   (symbol (lib_id "HPS:VCC") (at 156.21 81.28 0) (unit 1)
     (in_bom yes) (on_board yes) (fields_autoplaced)
@@
     (pin "1")
   )
+  (symbol (lib_id "HPS:TestPoint") (at 100.33 166.37 0) (unit 1)
+    (in_bom yes) (on_board yes) (fields_autoplaced)
+    (property "Reference" "TP6" (id 0) (at 102.87 161.7979 0)
+      (effects (font (size 1.27 1.27)) (justify left))
+    )
+    (property "Value" "TestPoint" (id 1) (at 102.87 164.3379 0)
+      (effects (font (size 1.27 1.27)) (justify left))
+    )
+    (property "Footprint" "footprints:TestPoint_THTPad_D2.0mm_Drill1.0mm" (id 2) (at 105.41 166.37 0)
+      (effects (font (size 1.27 1.27)) hide)
+    )
+    (property "Datasheet" "~" (id 3) (at 105.41 166.37 0)
+      (effects (font (size 1.27 1.27)) hide)
+    )
+    (pin "1")
+  )
   (symbol (lib_id "HPS:GND") (at 118.11 207.01 0) (unit 1)
     (in_bom yes) (on_board yes) (fields_autoplaced)
@@
     (pin "2")
   )
+  (symbol (lib_id "HPS:TestPoint") (at 90.17 201.93 0) (unit 1)
+    (in_bom yes) (on_board yes) (fields_autoplaced)
+    (property "Reference" "TP4" (id 0) (at 92.71 197.3579 0)
+      (effects (font (size 1.27 1.27)) (justify left))
+    )
+    (property "Value" "TestPoint" (id 1) (at 92.71 199.8979 0)
+      (effects (font (size 1.27 1.27)) (justify left))
+    )
+    (property "Footprint" "footprints:TestPoint_THTPad_D2.0mm_Drill1.0mm" (id 2) (at 95.25 201.93 0)
+      (effects (font (size 1.27 1.27)) hide)
+    )
+    (property "Datasheet" "~" (id 3) (at 95.25 201.93 0)
+      (effects (font (size 1.27 1.27)) hide)
+    )
+    (pin "1")
+  )
   (symbol (lib_id "HPS:VCC") (at 196.85 81.28 0) (unit 1)
     (in_bom yes) (on_board yes) (fields_autoplaced)
@@
     (pin "2")
   )
+  (symbol (lib_id "HPS:TestPoint") (at 81.28 53.34 0) (unit 1)
+    (in_bom yes) (on_board yes) (fields_autoplaced)
+    (property "Reference" "TP2" (id 0) (at 83.82 48.7679 0)
+      (effects (font (size 1.27 1.27)) (justify left))
+    )
+    (property "Value" "TestPoint" (id 1) (at 83.82 51.3079 0)
+      (effects (font (size 1.27 1.27)) (justify left))
+    )
+    (property "Footprint" "footprints:TestPoint_THTPad_D2.0mm_Drill1.0mm" (id 2) (at 86.36 53.34 0)
+      (effects (font (size 1.27 1.27)) hide)
+    )
+    (property "Datasheet" "~" (id 3) (at 86.36 53.34 0)
+      (effects (font (size 1.27 1.27)) hide)
+    )
+    (pin "1")
+  )
   (symbol (lib_id "HPS:GND") (at 39.37 203.2 0) (unit 1)
     (in_bom yes) (on_board yes) (fields_autoplaced)
@@
     (pin "2")
   )
+  (symbol (lib_id "HPS:TestPoint") (at 99.06 147.32 0) (unit 1)
+    (in_bom yes) (on_board yes) (fields_autoplaced)
+    (property "Reference" "TP5" (id 0) (at 101.6 142.7479 0)
+      (effects (font (size 1.27 1.27)) (justify left))
+    )
+    (property "Value" "TestPoint" (id 1) (at 101.6 145.2879 0)
+      (effects (font (size 1.27 1.27)) (justify left))
+    )
+    (property "Footprint" "footprints:TestPoint_THTPad_D2.0mm_Drill1.0mm" (id 2) (at 104.14 147.32 0)
+      (effects (font (size 1.27 1.27)) hide)
+    )
+    (property "Datasheet" "~" (id 3) (at 104.14 147.32 0)
+      (effects (font (size 1.27 1.27)) hide)
+    )
+    (pin "1")
+  )
   (symbol (lib_id "HPS:VCC") (at 64.77 171.45 0) (unit 1)
     (in_bom yes) (on_board yes) (fields_autoplaced)
@@
       (reference "TP1") (unit 1) (value "TestPoint") (footprint "footprints:TestPoint_THTPad_D2.0mm_Drill1.0mm")
     )
+    (path "/806326c9-5c7d-4364-b071-ccbbf5b84f0b"
+      (reference "TP2") (unit 1) (value "TestPoint") (footprint "footprints:TestPoint_THTPad_D2.0mm_Drill1.0mm")
+    )
+    (path "/33cc36c9-040d-4fca-8c47-1dc3d15e1d51"
+      (reference "TP3") (unit 1) (value "TestPoint") (footprint "footprints:TestPoint_THTPad_D2.0mm_Drill1.0mm")
+    )
+    (path "/49d856ce-c6c7-49e6-9542-62e980e79699"
+      (reference "TP4") (unit 1) (value "TestPoint") (footprint "footprints:TestPoint_THTPad_D2.0mm_Drill1.0mm")
+    )
+    (path "/d64701d2-ae8c-47d7-81b2-028ac65343b7"
+      (reference "TP5") (unit 1) (value "TestPoint") (footprint "footprints:TestPoint_THTPad_D2.0mm_Drill1.0mm")
+    )
+    (path "/4550f668-63f3-493b-a2eb-feb398f97598"
+      (reference "TP6") (unit 1) (value "TestPoint") (footprint "footprints:TestPoint_THTPad_D2.0mm_Drill1.0mm")
+    )
     (path "/db21ff12-4369-4043-a00a-4a3e857a1efc"

Commit message: Pre Gerber Edits
Parts:
- removed TP2: TestPoint, footprints:TestPoint_THTPad_D2.0mm_Drill1.0mm, symbol HPS:TestPoint
- added J3: Conn_02x03_Odd_Even, footprints:PinHeader_2x03_P2.54mm_Vertical, symbol HPS:Conn_02x03_Odd_Even
Connections:
- net D4: now also U2.28 (PC5); no longer U2.17 (PB3)
- net GND: now also J3.6 (Pin_6)
- net RESET: now also J3.5 (Pin_5)
- net VCC: now also J3.2 (Pin_2)
- net MISO: now reaches U2.18 (PB4)
- net MISO: now also J3.1 (Pin_1)
- net ICSP_SCK: now reaches U2.19 (PB5)
- net ICSP_SCK: now also J3.3 (Pin_3)
- new net MOSI: J3.4 (Pin_4), U2.17 (PB3)
- no-connect marks 11 -> 8
Other:
- note added: "ICSP"
- moved on the sheet: BT1, R11, R12, U1, Y2
